File: Hardware/Qwiic Mux.brd (EAGLE design)
At the start: 40.6 x 54.6 mm, 77 parts, among them J1 SMD, J10 SMD, J11 PTH, J12 PTH, J13 PTH, J14 PTH, J2 SMD, J23 SMD, J24 SMD, J25 SMD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

Commit message: Fixing silk. Fixing 5V LED circuit.
Parts:
- added D3: 3.3V, SparkFun-DiscreteSemi:SOD-323
- R26: value 330 -> 1k
- renumbered R23 to R26
Connections:
- new net N$2: D3.C, R26.1
- net GND: now also D3.A; no longer R26.1
Routing:
- net N$2: track 0.00 -> 2.03 mm
Changed lines of the file:
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@@
 <text x="9.398" y="30.607" size="1.27" layer="21" font="vector" ratio="15" rot="R90" align="center">3.3V</text>
 <text x="9.398" y="20.447" size="1.27" layer="21" font="vector" ratio="15" rot="R90" align="center">2.8V</text>
-<text x="9.398" y="10.287" size="1.27" layer="21" font="vector" ratio="15" rot="SR90" align="center">5V</text>
+<text x="9.398" y="10.287" size="1.27" layer="21" font="vector" ratio="15" rot="SR90" align="center">VIN</text>
 <text x="36.195" y="39.37" size="1.016" layer="22" font="vector" ratio="15" rot="MR0" align="center">3.3V</text>
 <text x="23.749" y="52.07" size="1.016" layer="22" font="vector" ratio="15" rot="MR0" align="center">3.3V</text>
 <text x="17.272" y="52.07" size="1.016" layer="22" font="vector" ratio="15" rot="MR0" align="center">5V</text>
 <text x="20.193" y="50.292" size="1.016" layer="22" font="vector" ratio="15" rot="MR0" align="center">VIN SEL</text>
-<text x="31.242" y="10.033" size="1.27" layer="21" font="vector" ratio="15" rot="SR270" align="center">5V</text>
+<text x="31.242" y="10.033" size="1.27" layer="21" font="vector" ratio="15" rot="SR270" align="center">VIN</text>
 <text x="31.242" y="20.193" size="1.27" layer="21" font="vector" ratio="15" rot="SR270" align="center">2.8V</text>
 <text x="31.242" y="30.353" size="1.27" layer="21" font="vector" ratio="15" rot="SR270" align="center">3.3V</text>
@@
 <text x="36.195" y="13.97" size="1.016" layer="22" font="vector" ratio="15" rot="MR0" align="center">SCL4</text>
 <text x="36.195" y="6.35" size="1.016" layer="22" font="vector" ratio="15" rot="MR0" align="center">GND</text>
-<text x="36.195" y="8.89" size="1.016" layer="22" font="vector" ratio="15" rot="MR0" align="center">5V</text>
+<text x="36.195" y="8.89" size="1.016" layer="22" font="vector" ratio="15" rot="MR0" align="center">VIN</text>
 <text x="4.191" y="8.89" size="1.016" layer="22" font="vector" ratio="15" rot="MR0" align="center">SDA3</text>
 <text x="4.191" y="6.35" size="1.016" layer="22" font="vector" ratio="15" rot="MR0" align="center">SCL3</text>
 <text x="4.191" y="13.97" size="1.016" layer="22" font="vector" ratio="15" rot="MR0" align="center">GND</text>
-<text x="4.191" y="11.43" size="1.016" layer="22" font="vector" ratio="15" rot="MR0" align="center">5V</text>
+<text x="4.191" y="11.43" size="1.016" layer="22" font="vector" ratio="15" rot="MR0" align="center">VIN</text>
 <text x="4.191" y="19.05" size="1.016" layer="22" font="vector" ratio="15" rot="MR0" align="center">SDA2</text>
 <text x="4.191" y="16.51" size="1.016" layer="22" font="vector" ratio="15" rot="MR0" align="center">SCL2</text>
@@
 <attribute name="PROD_ID" value="DIO-08575" x="16.51" y="5.08" size="1.778" layer="27" font="vector" ratio="15" rot="R90" display="off"/>
 </element>
-<element name="R23" library="SparkFun-Resistors" package="0603" value="330" x="16.51" y="8.89" rot="R270">
-<attribute name="PROD_ID" value="RES-00818" x="16.51" y="8.89" size="1.778" layer="27" font="vector" ratio="15" rot="R270" display="off"/>
-</element>
 <element name="R25" library="SparkFun-Resistors" package="0603" value="330" x="24.13" y="8.89" rot="R270">
 <attribute name="PROD_ID" value="RES-00818" x="24.13" y="8.89" size="1.778" layer="27" font="vector" ratio="15" rot="R270" display="off"/>
@@
 <element name="R24" library="SparkFun-Resistors" package="0603" value="330" x="20.32" y="8.89" rot="R270">
 <attribute name="PROD_ID" value="RES-00818" x="20.32" y="8.89" size="1.778" layer="27" font="vector" ratio="15" rot="R270" display="off"/>
+</element>
+<element name="R26" library="SparkFun-Resistors" package="0603" value="1k" x="16.51" y="8.89" rot="R270">
+<attribute name="PROD_ID" value="RES-07856" x="16.51" y="8.89" size="1.778" layer="27" font="vector" ratio="15" rot="R270" display="off"/>
+</element>
+<element name="D3" library="SparkFun-DiscreteSemi" package="SOD-323" value="3.3V" x="18.415" y="8.89" rot="R270">
+<attribute name="PROD_ID" value="DIO-11284" x="18.415" y="8.89" size="1.778" layer="27" font="vector" ratio="15" rot="R270" display="off"/>
 </element>
 </elements>
@@
 <via x="24.13" y="41.91" extent="1-16" drill="0.381"/>
 <via x="20.32" y="24.13" extent="1-16" drill="0.381"/>
-<contactref element="R23" pad="1"/>
 <contactref element="R25" pad="1"/>
 <contactref element="R24" pad="1"/>
+<contactref element="D3" pad="A"/>
 </signal>
 <signal name="3.3V">
@@
 <signal name="N$4">
 <contactref element="D4" pad="C"/>
-<contactref element="R23" pad="2"/>
-<wire x1="16.51" y1="5.957" x2="16.51" y2="8.04" width="0.1778" layer="1"/>
+<contactref element="R26" pad="2"/>
+<wire x1="16.51" y1="8.04" x2="16.51" y2="5.957" width="0.1778" layer="1"/>
+</signal>
+<signal name="N$2">
+<contactref element="R26" pad="1"/>
+<contactref element="D3" pad="C"/>
+<wire x1="18.415" y1="10.04" x2="17.66" y2="10.04" width="0.1778" layer="1"/>
+<wire x1="17.66" y1="10.04" x2="17.36" y2="9.74" width="0.1778" layer="1"/>
+<wire x1="16.51" y1="9.74" x2="17.36" y2="9.74" width="0.1778" layer="1"/>
 </signal>
 </signals>
